Commit message: Update arm_links.xacro

File: src/sort_robotic_arm_description/urdf/arm_links.xacro (robot description, xacro)
@@ -3,5 +3,5 @@
     <link name="ground_link" />
     <xacro:cylinder_link name="base" file="package://sort_robotic_arm_description/meshes/Arm_Base/Base.STL"
-            radius="0.60625" length="0.56" color="yellow" xyz_visual="-0.60625 0.60625 0"
+            radius="0.60625" length="0.56" color="black" xyz_visual="-0.60625 0.60625 0"
             rpy_visual="1.57 0 0" xyz_collision="0 0 0.28" rpy_collision="0 0 0" mass="0.12115"
             ixx="0.16" ixy="0.0" ixz="0.0" iyy="0.17" iyz="0.0" izz="0.26" />
@@ -11,5 +11,5 @@
             ixx="0.018" ixy="0.0" ixz="0.0" iyy="0.01" iyz="0.0" izz="0.01" />
     <xacro:cylinder_link name="waist" file="package://sort_robotic_arm_description/meshes/Arm_Base/Waist.STL"
-            radius="0.485" length="0.16" color="yellow" xyz_visual="-0.485 -0.485 0"
+            radius="0.485" length="0.16" color="black" xyz_visual="-0.485 -0.485 0"
             rpy_visual="0 0 0" xyz_collision="0 0 0.08" rpy_collision="0 0 0" mass="0.09702"
             ixx="0.085" ixy="0.0" ixz="-0.003" iyy="0.0006" iyz="-0.008" izz="0.07" />
@@ -19,5 +19,5 @@
             ixx="0.018" ixy="0.0" ixz="0.0" iyy="0.01" iyz="0.0" izz="0.01" />
     <xacro:cylinder_link name="arm1" file="package://sort_robotic_arm_description/meshes/Arm_Base/Arm1.STL"
-            radius="0.21" length="1.62" color="yellow" xyz_visual="0.3125 0.21 -0.23"
+            radius="0.21" length="1.62" color="black" xyz_visual="0.3125 0.21 -0.23"
             rpy_visual="0 0 -3.14" xyz_collision="0.025 -0.63 -0.05" rpy_collision="1.57 0 0" mass="0.05231"
             ixx="0.01" ixy="0.0" ixz="0.0" iyy="0.00006" iyz="0.0" izz="0.01" />
@@ -27,5 +27,5 @@
             ixx="0.018" ixy="0.0" ixz="0.0" iyy="0.01" iyz="0.0" izz="0.01" />
     <xacro:box_link name="arm2" file="package://sort_robotic_arm_description/meshes/Arm_Base/Arm2.STL"
-            size="0.38 1.15 0.27" color="yellow" xyz_visual="-0.19 -0.2525 -0.242"
+            size="0.38 1.15 0.27" color="black" xyz_visual="-0.19 -0.2525 -0.242"
             rpy_visual="0 0 0" xyz_collision="0 0.35 -0.135" rpy_collision="0 0 0" mass="0.05161"
             ixx="0.00058" ixy="0.0" ixz="0.0" iyy="0.00009" iyz="0.0" izz="0.00062" />
@@ -35,5 +35,5 @@
             ixx="0.000013" ixy="0.0" ixz="0.0" iyy="0.00008" iyz="0.0" izz="0.00008" />
     <xacro:box_link name="arm3" file="package://sort_robotic_arm_description/meshes/Arm_Base/Arm3.STL"
-            size="0.28 0.33 0.46" color="yellow" xyz_visual="-0.14 0 0.215"
+            size="0.28 0.33 0.46" color="black" xyz_visual="-0.14 0 0.215"
             rpy_visual="-1.57 0 0" xyz_collision="0 0.2 0" rpy_collision="-1.57 0 0" mass="0.0206"
             ixx="0.000063" ixy="0.0" ixz="0.000007" iyy="0.00005" iyz="0.0" izz="0.000032" />
@@ -43,5 +43,5 @@
             ixx="0.000013" ixy="0.0" ixz="0.0" iyy="0.00008" iyz="0.0" izz="0.00008" />
     <xacro:box_link name="gripper_base" file="package://sort_robotic_arm_description/meshes/Arm_Gripper/Gripper_Base.STL"
-            size="0.533 0.77 0.24" color="yellow" xyz_visual="-0.14 -0.63 -0.14"
+            size="0.533 0.77 0.24" color="black" xyz_visual="-0.14 -0.63 -0.14"
             rpy_visual="0 0 0" xyz_collision="0.1 -0.28 0" rpy_collision="0 0 0" mass="0.02131"
             ixx="0.00009" ixy="0.000025" ixz="0.0000055" iyy="0.00005" iyz="0.000016" izz="0.00012" />
@@ -51,9 +51,9 @@
             ixx="0.000013" ixy="0.0" ixz="0.0" iyy="0.00008" iyz="0.0" izz="0.00008" />
     <xacro:cylinder_link name="gear2" file="package://sort_robotic_arm_description/meshes/Arm_Gripper/Gear2.STL"
-            radius="0.133" length="0.04" color="yellow" xyz_visual="0.1209 -0.3475 0"
+            radius="0.133" length="0.04" color="black" xyz_visual="0.1209 -0.3475 0"
             rpy_visual="0 -1.57 0" xyz_collision="-0.01 0 0" rpy_collision="0 0 0" mass="0.00277"
             ixx="0.00005" ixy="0.0" ixz="0.0" iyy="0.0001" iyz="0.0" izz="0.000046" />
     <xacro:cylinder_link name="gear1" file="package://sort_robotic_arm_description/meshes/Arm_Gripper/Gear1.STL"
-            radius="0.133" length="0.04" color="yellow" xyz_visual="0.1209 -0.1463 0"
+            radius="0.133" length="0.04" color="black" xyz_visual="0.1209 -0.1463 0"
             rpy_visual="0 -1.57 0" xyz_collision="-0.01 0 0" rpy_collision="0 0 0" mass="0.00332"
             ixx="0.00005" ixy="0.0" ixz="0.0" iyy="0.0001" iyz="0.0" izz="0.000046" />
@@ -65,5 +65,5 @@
                 </geometry>
                 <origin xyz="0.04 0.04 0" rpy="0 0 3.14" />
-                <material name="yellow" />
+                <material name="black" />
             </visual>
             <collision>
@@ -93,5 +93,5 @@
                 </geometry>
                 <origin xyz="${xyz_visual}" rpy="${rpy}" />
-                <material name="yellow" />
+                <material name="black" />
             </visual>
             <collision>
